Commit message: spawning robot with realsense RGBD cam (lowFPS)

File: camera_description/urdf/robots/robot_3d.urdf.xacro (robot description, xacro)
@@ -1,4 +1,4 @@
 <?xml version="1.0"?>
-<robot xmlns:xacro="http://www.ros.org/wiki/xacro" name="robot_3d">
+<robot name="robot_3d" xmlns:xacro="http://www.ros.org/wiki/xacro" xmlns:gz="http://gazebosim.org/schema">
     <xacro:property name="M_PI" value="3.1415926535897931" />
     <xacro:arg name="robot_name" default="robot_3d"/>
@@ -8,4 +8,5 @@
     <xacro:include filename="$(find camera_description)/urdf/mech/mecanum_wheel.urdf.xacro"/>
     <xacro:include filename="$(find camera_description)/urdf/sensors/rgbd_camera.urdf.xacro"/>
+    <xacro:include filename="$(find camera_description)/urdf/control/camera_control.gazebo"/>
     <xacro:robot_3d_base prefix="$(arg prefix)"/>
     <xacro:mecanum_wheel
@@ -34,15 +35,102 @@
       xyz_offset="0.105 0 0.03"
       rpy_offset="0 0 0"/>
-    <!--
-    <xacro:include filename="$(find mec_mobile_description)/urdf/control/velocity_control_plugin.urdf.xacro" />
-    <xacro:load_velocity_control_plugin use_gazebo="$(arg use_gazebo)"/>
-    <xacro:include filename="$(find mec_mobile_description)/urdf/control/gazebo_sim_ros2_control.urdf.xacro" />
-    <xacro:load_gazebo_sim_ros2_control_plugin
-      robot_name="$(arg robot_name)"
-      use_gazebo="$(arg use_gazebo)"/>
-    <xacro:include filename="$(find mec_mobile_description)/urdf/control/robot_3d_ros2_control.urdf.xacro" />
-    <xacro:mec_mobile_ros2_control
-      prefix="$(arg prefix)"
-      use_gazebo="$(arg use_gazebo)"/>
-    -->
+    <!-- 2.4 add Gazebo frictions -->
+    <gazebo reference='front_left_wheel_link'>
+      <collision>
+        <surface>
+          <friction>
+            <ode>
+              <mu>1.5</mu>
+              <mu2>0.0</mu2>
+              <fdir1 gz:expressed_in="base_footprint">1 -1 0</fdir1>
+            </ode>
+          </friction>
+        </surface>
+      </collision>
+    </gazebo>
+    <gazebo reference='back_left_wheel_link'>
+      <collision>
+        <surface>
+          <friction>
+            <ode>
+              <mu>1.5</mu>
+              <mu2>0.0</mu2>
+              <fdir1 gz:expressed_in="base_footprint">1 1 0</fdir1>
+            </ode>
+          </friction>
+        </surface>
+      </collision>
+    </gazebo>
+    <gazebo reference='front_right_wheel_link'>
+      <collision>
+        <surface>
+          <friction>
+            <ode>
+              <mu>1.5</mu>
+              <mu2>0.0</mu2>
+              <fdir1 gz:expressed_in="base_footprint">1 1 0</fdir1>
+            </ode>
+          </friction>
+        </surface>
+      </collision>
+    </gazebo>
+    <gazebo reference='back_right_wheel_link'>
+      <collision>
+        <surface>
+          <friction>
+            <ode>
+              <mu>1.5</mu>
+              <mu2>0.0</mu2>
+              <fdir1 gz:expressed_in="base_footprint">1 -1 0</fdir1>
+            </ode>
+          </friction>
+        </surface>
+      </collision>
+    </gazebo>
+    <gazebo reference="base_link">
+      <mu1>0.000002</mu1>
+      <mu2>0.000002</mu2>
+      <!-- <material>Gazebo/Red</material> -->
+    </gazebo>
+    <!-- 2.5.1 Camera physical properties -->
+    <!-- <joint type="fixed" name="camera_joint">
+      <origin xyz="0.092 0 0.05" rpy="0 0 0"/>
+      <child link="camera_link"/>
+      <parent link="base_link"/>
+      <axis xyz="0 1 0" />
+    </joint>
+    <link name='camera_link'>
+      <pose>0 0 0 0 0 0</pose>
+      <inertial>
+        <mass value="0.1"/>
+        <origin xyz="0 0 0" rpy="0 0 0"/>
+        <inertia
+            ixx="1e-6" ixy="0" ixz="0"
+            iyy="1e-6" iyz="0"
+            izz="1e-6"/>
+      </inertial>
+      <collision name='collision'>
+        <origin xyz="0 0 0" rpy="0 0 0"/>
+        <geometry>
+          <box size=".03 .03 .03"/>
+        </geometry>
+      </collision>
+      <visual name='camera_link_visual'>
+        <origin xyz="0 0 0" rpy="0 0 0"/>
+        <geometry>
+          <box size=".02 .02 .02"/>
+        </geometry>
+      </visual>
+    </link>
+    <gazebo reference="camera_link">
+      <material>Gazebo/Red</material>
+    </gazebo>
+    <joint type="fixed" name="camera_optical_joint">
+      <origin xyz="0 0 0" rpy="-1.5707 0 -1.5707"/>
+      <child link="camera_link_optical"/>
+      <parent link="camera_link"/>
+    </joint>
+    <link name="camera_link_optical">
+    </link> -->
+    <!-- 2.5.1 End -->
 </robot>

Commit message: box+camera spawned in rviz

File: camera_description/urdf/robots/robot_3d.urdf.xacro (robot description, xacro)
@@ -1,136 +1,38 @@
 <?xml version="1.0"?>
-<robot name="robot_3d" xmlns:xacro="http://www.ros.org/wiki/xacro" xmlns:gz="http://gazebosim.org/schema">
-    <xacro:property name="M_PI" value="3.1415926535897931" />
-    <xacro:arg name="robot_name" default="robot_3d"/>
-    <xacro:arg name="prefix" default=""/>
-    <xacro:arg name="use_gazebo" default="false"/>
-    <xacro:include filename="$(find camera_description)/urdf/mech/robot_3d_base.urdf.xacro"/>
-    <xacro:include filename="$(find camera_description)/urdf/mech/mecanum_wheel.urdf.xacro"/>
-    <xacro:include filename="$(find camera_description)/urdf/sensors/rgbd_camera.urdf.xacro"/>
-    <xacro:include filename="$(find camera_description)/urdf/control/camera_control.gazebo"/>
-    <xacro:robot_3d_base prefix="$(arg prefix)"/>
-    <xacro:mecanum_wheel
-      prefix="$(arg prefix)"
-      side="front_left"
-      x_reflect="1"
-      y_reflect="1"/>
-    <xacro:mecanum_wheel
-      prefix="$(arg prefix)"
-      side="front_right"
-      x_reflect="1"
-      y_reflect="-1"/>
-    <xacro:mecanum_wheel
-      prefix="$(arg prefix)"
-      side="back_left"
-      x_reflect="-1"
-      y_reflect="1"/>
-    <xacro:mecanum_wheel
-      prefix="$(arg prefix)"
-      side="back_right"
-      x_reflect="-1"
-      y_reflect="-1"/>
-    <xacro:rgbd_camera
-      prefix="$(arg prefix)"
-      camera_name="cam_1"
-      xyz_offset="0.105 0 0.03"
-      rpy_offset="0 0 0"/>
-    <!-- 2.4 add Gazebo frictions -->
-    <gazebo reference='front_left_wheel_link'>
-      <collision>
-        <surface>
-          <friction>
-            <ode>
-              <mu>1.5</mu>
-              <mu2>0.0</mu2>
-              <fdir1 gz:expressed_in="base_footprint">1 -1 0</fdir1>
-            </ode>
-          </friction>
-        </surface>
-      </collision>
-    </gazebo>
-    <gazebo reference='back_left_wheel_link'>
-      <collision>
-        <surface>
-          <friction>
-            <ode>
-              <mu>1.5</mu>
-              <mu2>0.0</mu2>
-              <fdir1 gz:expressed_in="base_footprint">1 1 0</fdir1>
-            </ode>
-          </friction>
-        </surface>
-      </collision>
-    </gazebo>
-    <gazebo reference='front_right_wheel_link'>
-      <collision>
-        <surface>
-          <friction>
-            <ode>
-              <mu>1.5</mu>
-              <mu2>0.0</mu2>
-              <fdir1 gz:expressed_in="base_footprint">1 1 0</fdir1>
-            </ode>
-          </friction>
-        </surface>
-      </collision>
-    </gazebo>
-    <gazebo reference='back_right_wheel_link'>
-      <collision>
-        <surface>
-          <friction>
-            <ode>
-              <mu>1.5</mu>
-              <mu2>0.0</mu2>
-              <fdir1 gz:expressed_in="base_footprint">1 -1 0</fdir1>
-            </ode>
-          </friction>
-        </surface>
-      </collision>
-    </gazebo>
-    <gazebo reference="base_link">
-      <mu1>0.000002</mu1>
-      <mu2>0.000002</mu2>
-      <!-- <material>Gazebo/Red</material> -->
-    </gazebo>
-    <!-- 2.5.1 Camera physical properties -->
-    <!-- <joint type="fixed" name="camera_joint">
-      <origin xyz="0.092 0 0.05" rpy="0 0 0"/>
-      <child link="camera_link"/>
-      <parent link="base_link"/>
-      <axis xyz="0 1 0" />
-    </joint>
-    <link name='camera_link'>
-      <pose>0 0 0 0 0 0</pose>
-      <inertial>
-        <mass value="0.1"/>
-        <origin xyz="0 0 0" rpy="0 0 0"/>
-        <inertia
-            ixx="1e-6" ixy="0" ixz="0"
-            iyy="1e-6" iyz="0"
-            izz="1e-6"/>
-      </inertial>
-      <collision name='collision'>
-        <origin xyz="0 0 0" rpy="0 0 0"/>
-        <geometry>
-          <box size=".03 .03 .03"/>
-        </geometry>
-      </collision>
-      <visual name='camera_link_visual'>
-        <origin xyz="0 0 0" rpy="0 0 0"/>
-        <geometry>
-          <box size=".02 .02 .02"/>
-        </geometry>
-      </visual>
-    </link>
-    <gazebo reference="camera_link">
-      <material>Gazebo/Red</material>
-    </gazebo>
-    <joint type="fixed" name="camera_optical_joint">
-      <origin xyz="0 0 0" rpy="-1.5707 0 -1.5707"/>
-      <child link="camera_link_optical"/>
-      <parent link="camera_link"/>
-    </joint>
-    <link name="camera_link_optical">
-    </link> -->
-    <!-- 2.5.1 End -->
+<robot name="robot_3d"
+  xmlns:xacro="http://www.ros.org/wiki/xacro"
+  xmlns:gz="http://gazebosim.org/schema">
+  <xacro:property name="M_PI" value="3.1415926535897931" />
+  <xacro:arg name="robot_name" default="robot_3d"/>
+  <xacro:arg name="prefix" default=""/>
+  <xacro:arg name="use_gazebo" default="false"/>
+  <xacro:include filename="$(find camera_description)/urdf/sensors/rgbd_camera.urdf.xacro"/>
+  <xacro:include filename="$(find camera_description)/urdf/control/camera_control.gazebo"/>
+  <xacro:rgbd_camera prefix="$(arg prefix)" camera_name="cam_1" xyz_offset="0.105 0 0.03" rpy_offset="0 0 0" material_color="0.5 0.2 0.2 1" />
+  <link name="base_link">
+    <!-- <inertial>
+      <mass value="1.0"/>
+      <origin xyz="0 0 0" rpy="0 0 0"/>
+      <inertia ixx="0.01" ixy="0" ixz="0" iyy="0.01" iyz="0" izz="0.01"/>
+    </inertial> -->
+    <collision>
+      <origin xyz="0 0 0" rpy="0 0 0"/>
+      <geometry>
+        <box size="0.1 0.2 0.1"/>
+      </geometry>
+    </collision>
+    <visual>
+      <origin xyz="0 0 0" rpy="0 0 0"/>
+      <geometry>
+        <box size="0.1 0.2 0.1"/>
+      </geometry>
+      <material name="red">
+        <color rgba="1 0.2 0.2 1.0"/>
+      </material>
+    </visual>
+  </link>
+  <gazebo reference="camera_link">
+    <material>Gazebo/Red</material>
+  </gazebo>
+  <!-- 2.5.1 End -->
 </robot>

File: camera_description/urdf/sensors/rgbd_camera.urdf.xacro (robot description, xacro)
@@ -73,5 +73,5 @@
       <child link="${prefix}${camera_name}_color_frame" />
     </joint>
-    <link name="${prefix}${camera_n</robot>ame}_color_frame"/>
+    <link name="${prefix}${camera_name}_color_frame"/>
     <joint name="${prefix}${camera_name}_color_optical_joint" type="fixed">
       <origin xyz="${optical_xyz_offset}" rpy="${optical_rpy_offset}" />

Commit message: fix camera positioning and gravity

File: camera_description/urdf/robots/robot_3d.urdf.xacro (robot description, xacro)
@@ -9,15 +9,21 @@
   <xacro:include filename="$(find camera_description)/urdf/sensors/rgbd_camera.urdf.xacro"/>
   <xacro:include filename="$(find camera_description)/urdf/control/camera_control.gazebo"/>
-  <xacro:rgbd_camera prefix="$(arg prefix)" camera_name="cam_1" xyz_offset="0.105 0 0.03" rpy_offset="0 0 0" material_color="0.5 0.2 0.2 1" />
+  <!-- Define box dimensions as variables -->
+  <xacro:property name="box_length" value="0.15" />
+  <xacro:property name="box_width" value="0.1" />
+  <xacro:property name="box_height" value="0.05" />
+  <!-- Define camera placement properties -->
+  <xacro:property name="camera_z_offset" value="0" />
+  <xacro:property name="camera_x_offset" value="0" />
+  <xacro:property name="camera_y_offset" value="${box_width/2+0.02}" /> <!-- add 2cm offset form camera origin -->
+  <xacro:property name="camera_rx_offset" value="0" />
+  <xacro:property name="camera_ry_offset" value="0" />
+  <xacro:property name="camera_rz_offset" value="${3.14/2}" />
+  <xacro:rgbd_camera prefix="$(arg prefix)" mass = "0.01" camera_name="cam_1" xyz_offset="${camera_x_offset} ${camera_y_offset} ${camera_z_offset}" rpy_offset="${camera_rx_offset} ${camera_ry_offset} ${camera_rz_offset}" material_color="0.5 0.2 0.2 1" />
   <link name="base_link">
-    <!-- <inertial>
-      <mass value="1.0"/>
-      <origin xyz="0 0 0" rpy="0 0 0"/>
-      <inertia ixx="0.01" ixy="0" ixz="0" iyy="0.01" iyz="0" izz="0.01"/>
-    </inertial> -->
     <collision>
       <origin xyz="0 0 0" rpy="0 0 0"/>
       <geometry>
-        <box size="0.1 0.2 0.1"/>
+        <box size="${box_length} ${box_width} ${box_height}"/>
       </geometry>
     </collision>
@@ -25,5 +31,5 @@
       <origin xyz="0 0 0" rpy="0 0 0"/>
       <geometry>
-        <box size="0.1 0.2 0.1"/>
+        <box size="${box_length} ${box_width} ${box_height}"/>
       </geometry>
       <material name="red">
@@ -32,6 +38,10 @@
     </visual>
   </link>
+  <gazebo reference="base_link">
+    <gravity>0</gravity>
+  </gazebo>
   <gazebo reference="camera_link">
     <material>Gazebo/Red</material>
+    <gravity>0</gravity>
   </gazebo>
   <!-- 2.5.1 End -->

Commit message: broadcasted camera, depth. and PC

File: camera_description/urdf/robots/robot_3d.urdf.xacro (robot description, xacro)
@@ -16,10 +16,28 @@
   <xacro:property name="camera_z_offset" value="0" />
   <xacro:property name="camera_x_offset" value="0" />
-  <xacro:property name="camera_y_offset" value="${box_width/2+0.02}" /> <!-- add 2cm offset form camera origin -->
+  <xacro:property name="camera_y_offset" value="${box_width/2+0.02}" />
+  <!-- add 2cm offset form camera origin -->
   <xacro:property name="camera_rx_offset" value="0" />
   <xacro:property name="camera_ry_offset" value="0" />
   <xacro:property name="camera_rz_offset" value="${3.14/2}" />
-  <xacro:rgbd_camera prefix="$(arg prefix)" mass = "0.01" camera_name="cam_1" xyz_offset="${camera_x_offset} ${camera_y_offset} ${camera_z_offset}" rpy_offset="${camera_rx_offset} ${camera_ry_offset} ${camera_rz_offset}" material_color="0.5 0.2 0.2 1" />
+  <xacro:rgbd_camera prefix="$(arg prefix)" mass = "0.01" camera_name="camera" xyz_offset="${camera_x_offset} ${camera_y_offset} ${camera_z_offset}" rpy_offset="${camera_rx_offset} ${camera_ry_offset} ${camera_rz_offset}" material_color="0.5 0.2 0.2 1" />
+  <!-- Define the new root link (dummy_link) -->
+  <link name="dummy_link">
+    <visual>
+      <geometry>
+        <box size="0.001 0.001 0.001"/>
+      </geometry>
+      <material name="transparent">
+        <color rgba="0 0 0 0"/>
+        <!-- Making it invisible -->
+      </material>
+    </visual>
+  </link>
   <link name="base_link">
+    <inertial>
+      <origin xyz="0 0 0" rpy="0 0 0"/>
+      <mass value="1.0"/>
+      <inertia ixx="0.1" ixy="0" ixz="0" iyy="0.1" iyz="0" izz="0.1"/>
+    </inertial>
     <collision>
       <origin xyz="0 0 0" rpy="0 0 0"/>
@@ -38,11 +56,50 @@
     </visual>
   </link>
+  <!-- Fixed joint connecting dummy_link to base_link -->
+  <joint name="dummy_to_base" type="fixed">
+    <parent link="dummy_link"/>
+    <child link="base_link"/>
+    <origin xyz="0 0 0" rpy="0 0 0"/>
+  </joint>
   <gazebo reference="base_link">
     <gravity>0</gravity>
   </gazebo>
+  <!-- STEP 7 - Camera -->
+  <!-- <joint type="fixed" name="camera_joint">
+    <origin xyz="${camera_x_offset} ${camera_y_offset} ${camera_z_offset}" rpy="${camera_rx_offset} ${camera_ry_offset} ${camera_rz_offset}"/>
+    <child link="camera_link"/>
+    <parent link="base_link"/>
+    <axis xyz="0 1 0" />
+  </joint>
+  <link name='camera_link'>
+    <pose>0 0 0 0 0 0</pose>
+    <inertial>
+      <mass value="0.1"/>
+      <origin xyz="0 0 0" rpy="0 0 0"/>
+      <inertia ixx="1e-6" ixy="0" ixz="0" iyy="1e-6" iyz="0" izz="1e-6" />
+    </inertial>
+    <collision name='collision'>
+      <origin xyz="0 0 0" rpy="0 0 0"/>
+      <geometry>
+        <box size=".03 .03 .03"/>
+      </geometry>
+    </collision>
+    <visual name='camera_link_visual'>
+      <origin xyz="0 0 0" rpy="0 0 0"/>
+      <geometry>
+        <box size=".03 .03 .03"/>
+      </geometry>
+    </visual>
+  </link> -->
   <gazebo reference="camera_link">
-    <material>Gazebo/Red</material>
-    <gravity>0</gravity>
+    <material>Gazebo/Blue</material>
   </gazebo>
+  <!-- <joint type="fixed" name="camera_optical_joint">
+    <origin xyz="0 0 0" rpy="-1.5707 0 -1.5707"/>
+    <child link="camera_link_optical"/>
+    <parent link="camera_link"/>
+  </joint>
+  <link name="camera_link_optical">
+  </link> -->
   <!-- 2.5.1 End -->
 </robot>

Commit message: spawned point plane and ibvs pipeline

File: camera_description/urdf/robots/robot_3d.urdf.xacro (robot description, xacro)
@@ -10,15 +10,15 @@
   <xacro:include filename="$(find camera_description)/urdf/control/camera_control.gazebo"/>
   <!-- Define box dimensions as variables -->
-  <xacro:property name="box_length" value="0.15" />
-  <xacro:property name="box_width" value="0.1" />
+  <xacro:property name="box_length" value="0.1" />
+  <xacro:property name="box_width" value="0.15" />
   <xacro:property name="box_height" value="0.05" />
   <!-- Define camera placement properties -->
   <xacro:property name="camera_z_offset" value="0" />
-  <xacro:property name="camera_x_offset" value="0" />
-  <xacro:property name="camera_y_offset" value="${box_width/2+0.02}" />
+  <xacro:property name="camera_x_offset" value="${box_length/2+0.02}" />
+  <xacro:property name="camera_y_offset" value="0" />
   <!-- add 2cm offset form camera origin -->
   <xacro:property name="camera_rx_offset" value="0" />
   <xacro:property name="camera_ry_offset" value="0" />
-  <xacro:property name="camera_rz_offset" value="${3.14/2}" />
+  <xacro:property name="camera_rz_offset" value="${0}" />
   <xacro:rgbd_camera prefix="$(arg prefix)" mass = "0.01" camera_name="camera" xyz_offset="${camera_x_offset} ${camera_y_offset} ${camera_z_offset}" rpy_offset="${camera_rx_offset} ${camera_ry_offset} ${camera_rz_offset}" material_color="0.5 0.2 0.2 1" />
   <!-- Define the new root link (dummy_link) -->

Commit message: backup before changing attaching camera to atmos

File: camera_description/urdf/robots/robot_3d.urdf.xacro (robot description, xacro)
@@ -68,41 +68,6 @@
     <gravity>0</gravity>
   </gazebo>
-  <!-- STEP 7 - Camera -->
-  <!-- <joint type="fixed" name="camera_joint">
-    <origin xyz="${camera_x_offset} ${camera_y_offset} ${camera_z_offset}" rpy="${camera_rx_offset} ${camera_ry_offset} ${camera_rz_offset}"/>
-    <child link="camera_link"/>
-    <parent link="base_link"/>
-    <axis xyz="0 1 0" />
-  </joint>
-  <link name='camera_link'>
-    <pose>0 0 0 0 0 0</pose>
-    <inertial>
-      <mass value="0.1"/>
-      <origin xyz="0 0 0" rpy="0 0 0"/>
-      <inertia ixx="1e-6" ixy="0" ixz="0" iyy="1e-6" iyz="0" izz="1e-6" />
-    </inertial>
-    <collision name='collision'>
-      <origin xyz="0 0 0" rpy="0 0 0"/>
-      <geometry>
-        <box size=".03 .03 .03"/>
-      </geometry>
-    </collision>
-    <visual name='camera_link_visual'>
-      <origin xyz="0 0 0" rpy="0 0 0"/>
-      <geometry>
-        <box size=".03 .03 .03"/>
-      </geometry>
-    </visual>
-  </link> -->
   <gazebo reference="camera_link">
     <material>Gazebo/Blue</material>
   </gazebo>
-  <!-- <joint type="fixed" name="camera_optical_joint">
-    <origin xyz="0 0 0" rpy="-1.5707 0 -1.5707"/>
-    <child link="camera_link_optical"/>
-    <parent link="camera_link"/>
-  </joint>
-  <link name="camera_link_optical">
-  </link> -->
-  <!-- 2.5.1 End -->
 </robot>

Commit message: testing xacro with atmos sdf

File: camera_description/urdf/robots/robot_3d.urdf.xacro (robot description, xacro)
@@ -21,5 +21,5 @@
   <xacro:property name="camera_ry_offset" value="0" />
   <xacro:property name="camera_rz_offset" value="${0}" />
-  <xacro:rgbd_camera prefix="$(arg prefix)" mass = "0.01" camera_name="camera" xyz_offset="${camera_x_offset} ${camera_y_offset} ${camera_z_offset}" rpy_offset="${camera_rx_offset} ${camera_ry_offset} ${camera_rz_offset}" material_color="0.5 0.2 0.2 1" />
+  <xacro:rgbd_camera prefix="$(arg prefix)" parent="dummy_link" mass = "0.01" camera_name="camera" xyz_offset="${camera_x_offset} ${camera_y_offset} ${camera_z_offset}" rpy_offset="${camera_rx_offset} ${camera_ry_offset} ${camera_rz_offset}" material_color="0.5 0.2 0.2 1" />
   <!-- Define the new root link (dummy_link) -->
   <link name="dummy_link">
@@ -35,5 +35,5 @@
     </visual>
   </link>
-  <link name="base_link">
+   <!--<link name="base_link">
     <gravity>0</gravity>
     <inertial>
@@ -58,5 +58,5 @@
     </visual>
   </link>
-  <!-- Fixed joint connecting dummy_link to base_link -->
+  <!~~> Fixed joint connecting dummy_link to base_link ~~>
   <joint name="dummy_to_base" type="fixed">
     <gravity>0</gravity>
@@ -64,8 +64,9 @@
     <child link="base_link"/>
     <origin xyz="0 0 0" rpy="0 0 0"/>
-  </joint>
+  </joint>-->
+<!--
   <gazebo reference="base_link">
     <gravity>0</gravity>
-  </gazebo>
+  </gazebo>-->
   <gazebo reference="camera_link">
     <material>Gazebo/Blue</material>
