Commit message: <feat> made new sdf for attaching atmos with camera link

File: camera_description/urdf/robots/robot_3d.urdf.xacro (robot description, xacro)
@@ -8,5 +8,4 @@
   <xacro:arg name="use_gazebo" default="false"/>
   <xacro:include filename="$(find camera_description)/urdf/sensors/rgbd_camera.urdf.xacro"/>
-  <xacro:include filename="$(find camera_description)/urdf/control/camera_control.gazebo"/>
   <!-- Define box dimensions as variables -->
   <xacro:property name="box_length" value="0.1" />
@@ -35,5 +34,5 @@
     </visual>
   </link>
-   <!--<link name="base_link">
+  <link name="base_link">
     <gravity>0</gravity>
     <inertial>
@@ -58,5 +57,5 @@
     </visual>
   </link>
-  <!~~> Fixed joint connecting dummy_link to base_link ~~>
+  <!--> Fixed joint connecting dummy_link to base_link -->
   <joint name="dummy_to_base" type="fixed">
     <gravity>0</gravity>
@@ -64,11 +63,59 @@
     <child link="base_link"/>
     <origin xyz="0 0 0" rpy="0 0 0"/>
-  </joint>-->
-<!--
+  </joint>
   <gazebo reference="base_link">
     <gravity>0</gravity>
-  </gazebo>-->
+  </gazebo>
+  <!-- Define sensor camera  -->
   <gazebo reference="camera_link">
     <material>Gazebo/Blue</material>
   </gazebo>
+  <gazebo>
+    <!-- use VelocityControl plugin -->
+    <plugin filename="gz-sim-velocity-control-system" name="gz::sim::systems::VelocityControl">
+      <topic>cmd_vel</topic>
+      <initial_linear>0 0 0</initial_linear>
+      <initial_angular>0 0 0</initial_angular>
+    </plugin>
+    <plugin filename="gz-sim-odometry-publisher-system" name="gz::sim::systems::OdometryPublisher">
+      <dimensions>3</dimensions>
+      <odom_topic>odom</odom_topic>
+      <odom_frame>odom</odom_frame>
+      <robot_base_frame>dummy_link</robot_base_frame>
+      <publish_tf>true</publish_tf>
+      <tf_topic>tf</tf_topic>
+      <odom_publish_frequency>30</odom_publish_frequency>
+      <xyz_offset>0 0 0</xyz_offset>
+      <rpy_offset>0 0 0</rpy_offset>
+    </plugin>
+  </gazebo>
+  <gazebo reference="camera_link">
+    <sensor name="rgbd_camera" type="rgbd_camera">
+      <camera>
+        <horizontal_fov>1.25</horizontal_fov>
+        <image>
+          <width>640</width>
+          <height>480</height>
+        </image>
+        <clip>
+          <near>0.3</near>
+          <far>15</far>
+        </clip>
+        <noise>
+          <type>gaussian</type>
+          <!-- Noise is sampled independently per pixel on each frame.
+               That pixel's noise value is added to each of its color
+               channels, which at that point lie in the range [0,1]. -->
+          <mean>0.0</mean>
+          <stddev>0.0025</stddev>
+        </noise>
+        <optical_frame_id>camera_link</optical_frame_id>
+      </camera>
+      <always_on>1</always_on>
+      <update_rate>30</update_rate>
+      <visualize>true</visualize>
+      <topic>camera</topic>
+      <gz_frame_id>camera_link</gz_frame_id>
+    </sensor>
+  </gazebo>
 </robot>
